File: hardware/vllink_lite.r3/vllink_lite.r3.sch (KiCad schematic (older format))
At the start: 43 parts, among them J1 USB_B_Mini, J2 Conn_01x05, J3 Conn_01x02, SW1 SW_Push, U1_LQFP48 GD32F350Cx, U1_QFN28 GD32F350Gx, U2 AP1117-33, U3 W25Q64

Commit message: layout vllink lite r3
Parts:
- C1, C2, C3, C4, C5, C6: footprint (none) -> Capacitor_SMD:C_0603_1608Metric
- FB1: footprint (none) -> Inductor_SMD:L_0603_1608Metric
- IO_A1, IO_B1: footprint (none) -> vllogic:PinSocket_1x5_P2.54mm_SMD
- J1: footprint (none) -> Connector_USB:USB_Mini-B_Lumberg_2486_01_Horizontal
- J2: footprint (none) -> Connector_PinHeader_2.54mm:PinHeader_1x05_P2.54mm_Vertical
- J3: footprint (none) -> Connector_PinHeader_2.54mm:PinHeader_1x02_P2.54mm_Vertical
- LED1: footprint (none) -> LED_THT:LED_D3.0mm-3
- R1, R10, R11, R12, R13, R14, R15, R16, R17, R2, R3, R4, R5, R6, R7, R8, R9: footprint (none) -> Resistor_SMD:R_0603_1608Metric
- SW1: footprint (none) -> vllogic:SW_PUSH_4.5mm_Hxx
- TP1, TP2, TP3, TP4, TP5, TP6, TP7, TP8: footprint (none) -> TestPoint:TestPoint_Pad_D1.0mm
- U1_LQFP48: footprint (none) -> Package_QFP:LQFP-48_7x7mm_P0.5mm
- U1_QFN28: footprint (none) -> vllogic:QFN-28-1EP_4x4mm_P0.4mm_EP2.7x2.7mm
Connections:
- no-connect marks 23 -> 27
