File: hardware/vllink_lite.r3/vllink_lite.r3.kicad_pcb (KiCad board)
At the start: 2 copper layers, 45.5 x 23.4 mm, 43 parts, among them J1 USB_B_Mini, J2 Conn_01x05, J3 Conn_01x02, SW1 SW_Push, U1_LQFP48 GD32F350Cx, U1_QFN28 GD32F350Gx, U2 AP1117-33, U3 W25Q64

Commit message: vllink_lite.r3 pcb finish
Parts:
- removed U1_QFN28: GD32F350Gx, vllogic:QFN-28-1EP_4x4mm_P0.4mm_EP2.7x2.7mm
- added G***: love_log, vllogic:love_log, B.Cu at (104.6, 113.2)
- added U1_28: GD32F350Gx, vllogic:QFN-28-1EP_4x4mm_P0.4mm_EP2.7x2.7mm, F.Cu at (115.8, 113.7)
- renumbered U1_LQFP48 to U1_48
