File: hardware/vllink_lite.r4.gd32e103cx/vllink_lite.r4.gd32e103cx.kicad_pcb (KiCad board)
At the start: 2 copper layers, 45.5 x 23.4 mm, 42 parts, among them J1 USB_B_Mini, J2 Conn_01x05, J3 Conn_01x02, SW1 SW_Push, U1_LQFP48 GD32E103Cx, U2 AP1117-33, U3 W25Q64

Commit message: vllink_lite.r4.gd32f350xx / vllink_lite.r4.gd32e103tx / vllink_lite.r4.gd32e103cx gerbers
Changed lines of the file:
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@@
   (layers
     (0 F.Cu signal)
-    (31 B.Cu signal)
+    (31 B.Cu signal hide)
     (32 B.Adhes user hide)
     (33 F.Adhes user hide)
@@
     (35 F.Paste user hide)
     (36 B.SilkS user hide)
-    (37 F.SilkS user hide)
+    (37 F.SilkS user)
     (38 B.Mask user)
     (39 F.Mask user hide)
@@
   )
   (setup
-    (last_trace_width 0.3048)
+    (last_trace_width 0.1016)
     (user_trace_width 0.1524)
     (user_trace_width 0.2032)
@@
     (pad_to_mask_clearance 0.051)
     (solder_mask_min_width 0.25)
-    (aux_axis_origin 88.392 99.314)
+    (aux_axis_origin 88.646 122.936)
     (grid_origin 88.392 99.314)
     (visible_elements 7FFFFFFF)
@@
     (tags "LQFP QFP")
     (attr smd)
-    (fp_text reference U1_LQFP48 (at 0 -5.85) (layer F.SilkS)
+    (fp_text reference U1_LQFP48 (at 0.635 -5.715) (layer F.SilkS)
       (effects (font (size 1 1) (thickness 0.15)))
     )
@@
     (tags resistor)
     (attr smd)
-    (fp_text reference R19 (at 0 -1.43) (layer F.SilkS)
+    (fp_text reference R19 (at 0 1.524) (layer F.SilkS)
       (effects (font (size 1 1) (thickness 0.15)))
     )
@@
     (tags resistor)
     (attr smd)
-    (fp_text reference R18 (at -1.524 -2.667 90) (layer F.SilkS)
+    (fp_text reference R18 (at -1.27 -1.524 90) (layer F.SilkS)
       (effects (font (size 1 1) (thickness 0.15)))
     )
@@
     (tags resistor)
     (attr smd)
-    (fp_text reference R16 (at 0 1.524) (layer F.SilkS)
+    (fp_text reference R16 (at 3.048 0) (layer F.SilkS)
       (effects (font (size 1 1) (thickness 0.15)))
     )
@@
     (at 129.54 106.172 180)
     (attr smd)
-    (fp_text reference IO_B1 (at 0.048 2.058 180) (layer B.SilkS)
+    (fp_text reference IO_B1 (at 0.048 2.058 180) (layer B.SilkS) hide
       (effects (font (size 1 1) (thickness 0.15)) (justify mirror))
     )
@@
     (at 129.54 106.172)
     (attr smd)
-    (fp_text reference IO_A1 (at 0 -2.058) (layer F.SilkS)
+    (fp_text reference IO_A1 (at 0 -2.058) (layer F.SilkS) hide
       (effects (font (size 1 1) (thickness 0.15)))
     )
@@
     (tags capacitor)
     (attr smd)
-    (fp_text reference C6 (at 2.032 2.921 90) (layer F.SilkS)
+    (fp_text reference C6 (at 0 -1.397 90) (layer F.SilkS)
       (effects (font (size 1 1) (thickness 0.15)))
     )
@@
     (tags capacitor)
     (attr smd)
-    (fp_text reference C5 (at 0 -1.43 45) (layer F.SilkS)
-      (effects (font (size 1 1) (thickness 0.15)))
-    )
+    (fp_text reference C5 (at 0 1.616446 45) (layer F.SilkS)
+      (effects (font (size 1 1) (thickness 0.15)))
+    )

Commit message: fix PCB text
Other:
- board text added: "TDI VCC TMS/SWDIO GND TCK/SWCLK TRST SRST/SWRST TXD TDO/SWO RXD"
- board text removed: "TDI VCC TMS/SWDIO GND TCK/SWCLK TSRT SRST/SWRST TXD TDO/SWO RXD"
Changed lines of the file:
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@@
   (gr_line (start 126.746 104.902) (end 115.57 104.902) (layer B.SilkS) (width 0.12))
   (gr_line (start 126.746 108.458) (end 126.746 104.902) (layer B.SilkS) (width 0.12))
-  (gr_text "TDI             VCC\nTMS/SWDIO    GND\nTCK/SWCLK    TSRT\nSRST/SWRST   TXD\nTDO/SWO      RXD" (at 126.492 111.252) (layer B.SilkS)
+  (gr_text "TDI             VCC\nTMS/SWDIO    GND\nTCK/SWCLK    TRST\nSRST/SWRST   TXD\nTDO/SWO      RXD" (at 126.492 111.252) (layer B.SilkS)
     (effects (font (size 1.6 0.7) (thickness 0.15)) (justify left mirror))
   )
