File: hardware/vllink_lite.r4.gd32f350xx/vllink_lite.r4.gd32f350xx.kicad_pcb (KiCad board)
At the start: 2 copper layers, 45.5 x 23.4 mm, 44 parts, among them J1 USB_B_Mini, J2 Conn_01x05, J3 Conn_01x02, SW1 SW_Push, U1_LQFP48 GD32F350Cx, U1_QFN28 GD32F350Gx, U2 AP1117-33, U3 W25Q64, NC

Commit message: vllink_lite.r4.gd32f350xx / vllink_lite.r4.gd32e103tx / vllink_lite.r4.gd32e103cx gerbers
Changed lines of the file:
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@@
     (pad_to_mask_clearance 0.051)
     (solder_mask_min_width 0.25)
-    (aux_axis_origin 88.392 99.314)
+    (aux_axis_origin 88.646 122.936)
     (grid_origin 88.392 99.314)
     (visible_elements 7FFFFFFF)
@@
     (at 129.54 106.172 180)
     (attr smd)
-    (fp_text reference IO_B1 (at 0.048 2.058 180) (layer B.SilkS)
+    (fp_text reference IO_B1 (at 0.048 2.058 180) (layer B.SilkS) hide
       (effects (font (size 1 1) (thickness 0.15)) (justify mirror))
     )
@@
     (at 129.54 106.172)
     (attr smd)
-    (fp_text reference IO_A1 (at 0 -2.058) (layer F.SilkS)
-      (effects (font (size 1 1) (thickness 0.15)))
-    )
+    (fp_text reference IO_A1 (at 0 -2.058) (layer F.SilkS) hide
+      (effects (font (size 1 1) (thickness 0.15)))
+    )

Commit message: fix PCB text
Other:
- board text added: "TDI VCC TMS/SWDIO GND TCK/SWCLK TRST SRST/SWRST TXD TDO/SWO RXD"
- board text removed: "TDI VCC TMS/SWDIO GND TCK/SWCLK TSRT SRST/SWRST TXD TDO/SWO RXD"
Changed lines of the file:
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@@
   (gr_line (start 126.746 104.902) (end 115.57 104.902) (layer B.SilkS) (width 0.12))
   (gr_line (start 126.746 108.458) (end 126.746 104.902) (layer B.SilkS) (width 0.12))
-  (gr_text "TDI             VCC\nTMS/SWDIO    GND\nTCK/SWCLK    TSRT\nSRST/SWRST   TXD\nTDO/SWO      RXD" (at 126.492 111.252) (layer B.SilkS)
+  (gr_text "TDI             VCC\nTMS/SWDIO    GND\nTCK/SWCLK    TRST\nSRST/SWRST   TXD\nTDO/SWO      RXD" (at 126.492 111.252) (layer B.SilkS)
     (effects (font (size 1.6 0.7) (thickness 0.15)) (justify left mirror))
   )
